Commit message: Updates to robot model

File: urdf/imports/builders.xacro (robot description, xacro)
@@ -188,4 +188,22 @@
             rpy="0 0 0"
             xyz="${0*scale} ${-79*scale} ${0*scale}" />
+        <link name="camera">
+            <visual>
+                <geometry>
+                    <box size="0.02 0.03 0.001"/> <!-- Simple box representation -->
+                </geometry>
+                <material name="RED" />
+            </visual>
+            <collision>
+                <geometry>
+                    <box size="0.03 0.03 0.001"/>
+                </geometry>
+            </collision>
+        </link>
+        <xacro:create_fixed_joint
+            parent="nose_chassis"
+            child="camera"
+            rpy="${-pi*7/12} 0 0"
+            xyz="${0*scale} ${0*scale} ${0*scale}" />
     </xacro:macro>
     <!-- Leg builder -->
