Commit message: Moved meshes into renamed model package

File: model/imports/parts.xacro (robot description, xacro)
@@ -2,5 +2,5 @@
 <robot xmlns:xacro="http://www.ros.org/wiki/xacro" name="Subwoofer_parts">
     <xacro:include filename="$(find subwoofer_model)/urdf/imports/constants.xacro"/>
-    <xacro:property name="parts_location" value="file://$(find subwoofer_model)/meshes"/>
+    <xacro:property name="parts_location" value="meshes"/>
     <!-- Servo -->
     <xacro:property name="servo_mesh" value="${parts_location}/Servo.dae" />
