Commit message: Reflected directory rename in robot file

File: model/imports/builders.xacro (robot description, xacro)
@@ -1,6 +1,6 @@
 <?xml version="1.0" encoding="UTF-8"?>
 <robot xmlns:xacro="http://www.ros.org/wiki/xacro" name="Subwoofer_builders">
-    <xacro:include filename="$(find subwoofer_model)/urdf/imports/constants.xacro"/>
-    <xacro:include filename="$(find subwoofer_model)/urdf/imports/materials.xacro"/>
+    <xacro:include filename="$(find subwoofer_model)/model/imports/constants.xacro"/>
+    <xacro:include filename="$(find subwoofer_model)/model/imports/materials.xacro"/>
     <!-- Link builder -->
     <xacro:macro name="create_link" params="name mesh rpy xyz mass">
@@ -59,5 +59,5 @@
             <child link="${child}"/>
             <axis xyz="${axis}"/>
-            <limit effort="1000.0" lower="${lower}" upper="${upper}" velocity="${velocity}"/>
+            <limit effort="1.0" lower="${lower}" upper="${upper}" velocity="${velocity}"/>
             <origin rpy="${rpy}" xyz="${xyz}"/>
             <dynamics damping="0.05" friction="0.05"/>
@@ -76,5 +76,5 @@
             parent="base_link"
             child="baseplate"
-            rpy="0 0 0"
+            rpy="0 0 -${pi/2}"
             xyz="0 0 0" />
         <xacro:create_link
@@ -209,4 +209,106 @@
     <!-- Leg builder -->
     <xacro:macro name="create_left_leg" params="parent name xyz">
+        <xacro:create_link
+            name="${name}_hip_servo"
+            mesh="${servo_mesh}"
+            xyz="${servo_xyz}"
+            rpy="${servo_rpy}"
+            mass="${servo_mass}" />
+        <xacro:create_revolute_joint
+            parent="${parent}"
+            child="${name}_hip_servo"
+            axis="-1 0 0"
+            lower="-0.78"
+            upper="0.78"
+            velocity="0.5"
+            rpy="0 0 -1.57075"
+            xyz="${xyz}" />
+        <xacro:create_link
+            name="${name}_hip"
+            mesh="${left_hind_mesh}"
+            xyz="${left_hind_xyz}"
+            rpy="${left_hind_rpy}"
+            mass="${left_hind_mass}" />
+        <xacro:create_fixed_joint
+            parent="${name}_hip_servo"
+            child="${name}_hip"
+            rpy="0 0 -1.57075"
+            xyz="${27.2*scale} ${-25*scale} ${-10*scale}" />
+        <xacro:create_link
+            name="${name}_midlimb_servo"
+            mesh="${servo_mesh}"
+            xyz="${servo_xyz}"
+            rpy="${servo_rpy}"
+            mass="${servo_mass}" />
+        <xacro:create_revolute_joint
+            parent="${name}_hip"
+            child="${name}_midlimb_servo"
+            axis="-1 0 0"
+            lower="-1.57"
+            upper="1.57"
+            velocity="0.5"
+            rpy="0 0 0"
+            xyz="0 0 0" />
+        <xacro:create_link
+            name="${name}_midlimb"
+            mesh="${left_midlimb_mesh}"
+            xyz="${left_midlimb_xyz}"
+            rpy="${left_midlimb_rpy}"
+            mass="${left_midlimb_mass}" />
+        <xacro:create_fixed_joint
+            parent="${name}_midlimb_servo"
+            child="${name}_midlimb"
+            rpy="0 0 -1.57075"
+            xyz="${9*scale} ${-13*scale} ${-107*scale}" />
+        <xacro:create_link
+            name="${name}_midlimb_cover"
+            mesh="${left_midlimb_cover_mesh}"
+            xyz="${left_midlimb_cover_xyz}"
+            rpy="${left_midlimb_cover_rpy}"
+            mass="${left_midlimb_cover_mass}" />
+        <xacro:create_fixed_joint
+            parent="${name}_midlimb"
+            child="${name}_midlimb_cover"
+            rpy="0 0 0"
+            xyz="0 ${49.7*scale} 0" />
+        <xacro:create_link
+            name="${name}_wrist_servo"
+            mesh="${servo_mesh}"
+            xyz="${servo_xyz}"
+            rpy="${servo_rpy}"
+            mass="${servo_mass}" />
+        <xacro:create_revolute_joint
+            parent="${name}_midlimb"
+            child="${name}_wrist_servo"
+            axis="-1 0 0"
+            lower="-${1/3*pi}"
+            upper="${4/5*pi}"
+            velocity="0.5"
+            rpy="0 0 1.57075"
+            xyz="0 0 0" />
+        <xacro:create_link
+            name="${name}_wrist"
+            mesh="${left_wrist_mesh}"
+            xyz="${left_wrist_xyz}"
+            rpy="${left_wrist_rpy}"
+            mass="${left_wrist_mass}" />
+        <xacro:create_fixed_joint
+            parent="${name}_wrist_servo"
+            child="${name}_wrist"
+            rpy="0 0 3.1415"
+            xyz="${53*scale} 0 0" />
+        <xacro:create_link
+            name="${name}_foot"
+            mesh="${foot_mesh}"
+            xyz="${foot_xyz}"
+            rpy="${foot_rpy}"
+            mass="${foot_mass}" />
+        <xacro:create_fixed_joint
+            parent="${name}_wrist"
+            child="${name}_foot"
+            rpy="${-pi/9} 0 0"
+            xyz="${26*scale} ${-6*scale} ${-135*scale}" />
+    </xacro:macro>
+    <xacro:macro name="create_right_leg" params="parent name xyz">
         <xacro:create_link
             name="${name}_hip_servo"
@@ -226,13 +328,13 @@
         <xacro:create_link
             name="${name}_hip"
-            mesh="${left_hind_mesh}"
-            xyz="${left_hind_xyz}"
-            rpy="${left_hind_rpy}"
-            mass="${left_hind_mass}" />
+            mesh="${right_hind_mesh}"
+            xyz="${right_hind_xyz}"
+            rpy="${right_hind_rpy}"
+            mass="${right_hind_mass}" />
         <xacro:create_fixed_joint
             parent="${name}_hip_servo"
             child="${name}_hip"
-            rpy="0 0 -1.57075"
-            xyz="${27.2*scale} ${-25*scale} ${-10*scale}" />
+            rpy="0 0 1.57075"
+            xyz="${27.2*scale} ${25*scale} ${-10*scale}" />
         <xacro:create_link
             name="${name}_midlimb_servo"
@@ -248,96 +350,5 @@
             upper="1.57"
             velocity="0.5"
-            rpy="0.8 0 0"
-            xyz="0 0 0" />
-        <xacro:create_link
-            name="${name}_midlimb"
-            mesh="${left_midlimb_mesh}"
-            xyz="${left_midlimb_xyz}"
-            rpy="${left_midlimb_rpy}"
-            mass="${left_midlimb_mass}" />
-        <xacro:create_fixed_joint
-            parent="${name}_midlimb_servo"
-            child="${name}_midlimb"
-            rpy="0 0 -1.57075"
-            xyz="${9*scale} ${-13*scale} ${-107*scale}" />
-        <xacro:create_link
-            name="${name}_midlimb_cover"
-            mesh="${left_midlimb_cover_mesh}"
-            xyz="${left_midlimb_cover_xyz}"
-            rpy="${left_midlimb_cover_rpy}"
-            mass="${left_midlimb_cover_mass}" />
-        <xacro:create_fixed_joint
-            parent="${name}_midlimb"
-            child="${name}_midlimb_cover"
-            rpy="0 0 0"
-            xyz="0 ${49.7*scale} 0" />
-        <xacro:create_link
-            name="${name}_wrist_servo"
-            mesh="${servo_mesh}"
-            xyz="${servo_xyz}"
-            rpy="${servo_rpy}"
-            mass="${servo_mass}" />
-        <xacro:create_revolute_joint
-            parent="${name}_midlimb"
-            child="${name}_wrist_servo"
-            axis="1 0 0"
-            lower="-2.6"
-            upper="1.1"
-            velocity="0.5"
-            rpy="-1.6 0 1.57075"
-            xyz="0 0 0" />
-        <xacro:create_link
-            name="${name}_wrist"
-            mesh="${left_wrist_mesh}"
-            xyz="${left_wrist_xyz}"
-            rpy="${left_wrist_rpy}"
-            mass="${left_wrist_mass}" />
-        <xacro:create_fixed_joint
-            parent="${name}_wrist_servo"
-            child="${name}_wrist"
-            rpy="0 0 3.1415"
-            xyz="${53*scale} 0 0" />
-    </xacro:macro>
-    <xacro:macro name="create_right_leg" params="parent name xyz">
-        <xacro:create_link
-            name="${name}_hip_servo"
-            mesh="${servo_mesh}"
-            xyz="${servo_xyz}"
-            rpy="${servo_rpy}"
-            mass="${servo_mass}" />
-        <xacro:create_revolute_joint
-            parent="${parent}"
-            child="${name}_hip_servo"
-            axis="1 0 0"
-            lower="-0.78"
-            upper="0.78"
-            velocity="0.5"
-            rpy="0 0 -1.57075"
-            xyz="${xyz}" />
-        <xacro:create_link
-            name="${name}_hip"
-            mesh="${right_hind_mesh}"
-            xyz="${right_hind_xyz}"
-            rpy="${right_hind_rpy}"
-            mass="${right_hind_mass}" />
-        <xacro:create_fixed_joint
-            parent="${name}_hip_servo"
-            child="${name}_hip"
-            rpy="0 0 1.57075"
-            xyz="${27.2*scale} ${25*scale} ${-10*scale}" />
-        <xacro:create_link
-            name="${name}_midlimb_servo"
-            mesh="${servo_mesh}"
-            xyz="${servo_xyz}"
-            rpy="${servo_rpy}"
-            mass="${servo_mass}" />
-        <xacro:create_revolute_joint
-            parent="${name}_hip"
-            child="${name}_midlimb_servo"
-            axis="1 0 0"
-            lower="-1.57"
-            upper="1.57"
-            velocity="0.5"
-            rpy="-0.8 0 0"
+            rpy="0 0 0"
             xyz="0 0 0" />
         <xacro:create_link
@@ -373,8 +384,8 @@
             child="${name}_wrist_servo"
             axis="1 0 0"
-            lower="-1.1"
-            upper="2.6"
+            lower="-${1/3*pi}"
+            upper="${4/5*pi}"
             velocity=".5"
-            rpy="1.6 0 1.57075"
+            rpy="0 0 1.57075"
             xyz="${0*scale} ${0*scale} ${0*scale}" />
         <xacro:create_link
@@ -389,4 +400,15 @@
             rpy="0 0 0"
             xyz="${53*scale} ${0*scale} ${0*scale}" />
+        <xacro:create_link
+            name="${name}_foot"
+            mesh="${foot_mesh}"
+            xyz="${foot_xyz}"
+            rpy="${foot_rpy}"
+            mass="${foot_mass}" />
+        <xacro:create_fixed_joint
+            parent="${name}_wrist"
+            child="${name}_foot"
+            rpy="${-pi/9} 0 0"
+            xyz="${-26.5*scale} ${-6*scale} ${-135*scale}" />
     </xacro:macro>
 </robot>

File: model/imports/materials.xacro (robot description, xacro)
@@ -1,5 +1,5 @@
 <?xml version="1.0" encoding="UTF-8"?>
 <robot xmlns:xacro="http://www.ros.org/wiki/xacro" name="Subwoofer_materials">
-    <xacro:include filename="$(find subwoofer_model)/urdf/imports/constants.xacro"/>
+    <xacro:include filename="$(find subwoofer_model)/model/imports/constants.xacro"/>
     <material name="BLACK">
         <color rgba="0.0 0.0 0.0 1.0"/>

File: model/imports/parts.xacro (robot description, xacro)
@@ -1,6 +1,6 @@
 <?xml version="1.0"?>
 <robot xmlns:xacro="http://www.ros.org/wiki/xacro" name="Subwoofer_parts">
-    <xacro:include filename="$(find subwoofer_model)/urdf/imports/constants.xacro"/>
-    <xacro:property name="parts_location" value="meshes"/>
+    <xacro:include filename="$(find subwoofer_model)/model/imports/constants.xacro"/>
+    <xacro:property name="parts_location" value="package://subwoofer_model/model/meshes"/>
     <!-- Servo -->
     <xacro:property name="servo_mesh" value="${parts_location}/Servo.dae" />
@@ -103,3 +103,8 @@
     <xacro:property name="right_wrist_rpy" value="0 1.57075 1.57075"/>
     <xacro:property name="right_wrist_mass" value="0.023"/>
+    <!-- Foot -->
+    <xacro:property name="foot_mesh" value="${parts_location}/V1.02_Foot.dae" />
+    <xacro:property name="foot_xyz" value="${165*scale} ${120*scale} ${80*scale}" />
+    <xacro:property name="foot_rpy" value="0 0 ${pi/2}"/>
+    <xacro:property name="foot_mass" value="0.010"/>
 </robot>

File: model/subwoofer.urdf.xacro (robot description, xacro)
@@ -1,23 +1,23 @@
 <?xml version="1.0"?>
 <robot xmlns:xacro="http://www.ros.org/wiki/xacro" name="Subwoofer">
-    <xacro:include filename="$(find subwoofer_model)/urdf/imports/constants.xacro"/>
-    <xacro:include filename="$(find subwoofer_model)/urdf/imports/parts.xacro"/>
-    <xacro:include filename="$(find subwoofer_model)/urdf/imports/builders.xacro"/>
+    <xacro:include filename="$(find subwoofer_model)/model/imports/constants.xacro"/>
+    <xacro:include filename="$(find subwoofer_model)/model/imports/parts.xacro"/>
+    <xacro:include filename="$(find subwoofer_model)/model/imports/builders.xacro"/>
     <xacro:create_body />
     <xacro:create_left_leg
         parent="front_outer_shoulder"
         name="front_left"
-        xyz="${-37*scale} ${0*scale} ${7*scale}" />
+        xyz="${-38*scale} ${0*scale} ${7*scale}" />
     <xacro:create_right_leg
         parent="front_outer_shoulder"
         name="front_right"
-        xyz="${37*scale} ${0*scale} ${7*scale}" />
+        xyz="${40*scale} ${0*scale} ${7*scale}" />
     <xacro:create_left_leg
         parent="back_inner_shoulder"
         name="back_left"
-        xyz="${-37*scale} ${0*scale} ${7*scale}" />
+        xyz="${-38*scale} ${0*scale} ${7*scale}" />
     <xacro:create_right_leg
         parent="back_inner_shoulder"
         name="back_right"
-        xyz="${37*scale} ${0*scale} ${7*scale}" />
+        xyz="${40*scale} ${0*scale} ${7*scale}" />
 </robot>

Commit message: Camera link name update

File: model/imports/builders.xacro (robot description, xacro)
@@ -188,5 +188,5 @@
             rpy="0 0 0"
             xyz="${0*scale} ${-79*scale} ${0*scale}" />
-        <link name="camera">
+        <link name="camera_link">
             <visual>
                 <geometry>
@@ -203,5 +203,5 @@
         <xacro:create_fixed_joint
             parent="nose_chassis"
-            child="camera"
+            child="camera_link"
             rpy="${-pi*7/12} 0 0"
             xyz="${0*scale} ${0*scale} ${0*scale}" />
